File: nob.kicad_sch (KiCad schematic)
At the start: 23 parts, among them U1 XIAO-ESP32-C3-SMD, U2 AS5600

Commit message: update
Parts:
- added C10, C11, C12, C13, C2, C3, C4, C5, C6, C7, C8, C9: 0.1uF, Capacitor_SMD:C_0805_2012Metric, symbol Device:C_Small
- added G10, G2, G3, G4, G7, G8, G9, P0, P1, P1.5, P10: Conn_01x01_Pin, Connector_Wire:SolderWire-0.1sqmm_1x01_D0.4mm_OD1mm, symbol Connector:Conn_01x01_Pin
- added R3: 500, Capacitor_SMD:C_0805_2012Metric, symbol Device:R_Small
- D1, D10, D11, D12, D2, D3, D4, D5, D6, D7, D8, D9: LCSC (none) -> C114586
- U2: LCSC (none) -> C499458
Connections:
- net +3.3V: now also P1.5.1 (Pin_1)
- net +5V: now also C10.2, C11.2, C12.2, C13.2, C2.2, C3.2, C4.2, C5.2, C6.2, C7.2, C8.2, C9.2, P1.1 (Pin_1)
- net GND: now also C10.1, C11.1, C12.1, C13.1, C2.1, C3.1, C4.1, C5.1, C6.1, C7.1, C8.1, C9.1, P0.1 (Pin_1), P10.1 (Pin_1)
- net LED: now also R3.1; no longer U1.1 (GPIO2_A0_D0)
- net at U1.10 (GPIO9_D9_MISO): now also G9.1 (Pin_1)
- net at U1.11 (GPIO10_D10_MOSI): now also G10.1 (Pin_1)
- net at U1.3 (GPIO4_A2_D2): now also G2.1 (Pin_1)
- net at U1.4 (GPIO5_A3_D3): now also G3.1 (Pin_1)
- net at U1.7 (GPIO21_D6_TX): now also G4.1 (Pin_1)
- net at U1.8 (GPIO20_D7_RX): now also G7.1 (Pin_1)
- net at U1.9 (GPIO8_D8_SCK): now also G8.1 (Pin_1)
- new net: R3.2, U1.1 (GPIO2_A0_D0)

Commit message: update
Parts:
- added LED_JUMP1, MAG_POWER1: Jumper_2_Bridged, Jumper:SolderJumper-2_P1.3mm_Bridged2Bar_Pad1.0x1.5mm, symbol Jumper:Jumper_2_Bridged
- BAT_N1, BAT_P1: footprint Connector_Wire:SolderWire-0.1sqmm_1x01_D0.4mm_OD1mm -> Connector_Wire:SolderWire-0.5sqmm_1x01_D0.9mm_OD2.1mm
Connections:
- net +5V: now also LED_JUMP1.2 (B), MAG_POWER1.1 (A); no longer C1.1, C10.2, C11.2, C12.2, C13.2, C2.2, C3.2, C4.2, C5.2, C6.2, C7.2, C8.2, C9.2, D1.1 (VDD), D10.1 (VDD), D11.1 (VDD), D12.1 (VDD), D2.1 (VDD), D3.1 (VDD), D4.1 (VDD), D5.1 (VDD), D6.1 (VDD), D7.1 (VDD), D8.1 (VDD), D9.1 (VDD), R1.1, R2.2, U2.1 (VDD5V)
- net BAT_P: now reaches BAT_P1.1 (Pin_1), U1.15 (BAT)
- new net: C1.1, MAG_POWER1.2 (B), R1.1, R2.2, U2.1 (VDD5V)
- new net LED_P: C10.2, C11.2, C12.2, C13.2, C2.2, C3.2, C4.2, C5.2, C6.2, C7.2, C8.2, C9.2, D1.1 (VDD), D10.1 (VDD), D11.1 (VDD), D12.1 (VDD), D2.1 (VDD), D3.1 (VDD), D4.1 (VDD), D5.1 (VDD), D6.1 (VDD), D7.1 (VDD), D8.1 (VDD), D9.1 (VDD), LED_JUMP1.1 (A)
Other:
- moved on the sheet: BAT_P1, R2
