File: nob.kicad_pcb (KiCad board)
At the start: 2 copper layers, 70 x 70.6 mm, 23 parts, among them U1 XIAO-ESP32-C3-SMD, U2 AS5600

Commit message: update
Parts:
- added C10: 0.1uF, Capacitor_SMD:C_0805_2012Metric, B.Cu at (119.7, 98.2)
- added C11: 0.1uF, Capacitor_SMD:C_0805_2012Metric, B.Cu at (135.2, 99.5)
- added C12: 0.1uF, Capacitor_SMD:C_0805_2012Metric, B.Cu at (149.3, 93.0)
- added C13: 0.1uF, Capacitor_SMD:C_0805_2012Metric, B.Cu at (158.2, 80.3)
- added C2: 0.1uF, Capacitor_SMD:C_0805_2012Metric, B.Cu at (159.5, 64.8)
- added C3: 0.1uF, Capacitor_SMD:C_0805_2012Metric, B.Cu at (153.0, 50.7)
- added C4: 0.1uF, Capacitor_SMD:C_0805_2012Metric, B.Cu at (140.3, 41.8)
- added C5: 0.1uF, Capacitor_SMD:C_0805_2012Metric, B.Cu at (124.8, 40.5)
- added C6: 0.1uF, Capacitor_SMD:C_0805_2012Metric, B.Cu at (110.7, 47.0)
- added C7: 0.1uF, Capacitor_SMD:C_0805_2012Metric, B.Cu at (101.8, 59.7)
- added C8: 0.1uF, Capacitor_SMD:C_0805_2012Metric, B.Cu at (100.5, 75.2)
- added C9: 0.1uF, Capacitor_SMD:C_0805_2012Metric, B.Cu at (107.0, 89.3)
- added G10: Conn_01x01_Pin, Connector_Wire:SolderWire-0.1sqmm_1x01_D0.4mm_OD1mm, F.Cu at (134.0, 57.2)
- added G2: Conn_01x01_Pin, Connector_Wire:SolderWire-0.1sqmm_1x01_D0.4mm_OD1mm, F.Cu at (122.0, 59.0)
- added G3: Conn_01x01_Pin, Connector_Wire:SolderWire-0.1sqmm_1x01_D0.4mm_OD1mm, F.Cu at (125.0, 61.8)
- added G4: Conn_01x01_Pin, Connector_Wire:SolderWire-0.1sqmm_1x01_D0.4mm_OD1mm, F.Cu at (125.0, 59.0)
- added G7: Conn_01x01_Pin, Connector_Wire:SolderWire-0.1sqmm_1x01_D0.4mm_OD1mm, F.Cu at (134.0, 60.0)
- added G8: Conn_01x01_Pin, Connector_Wire:SolderWire-0.1sqmm_1x01_D0.4mm_OD1mm, F.Cu at (137.0, 60.0)
- added G9: Conn_01x01_Pin, Connector_Wire:SolderWire-0.1sqmm_1x01_D0.4mm_OD1mm, F.Cu at (137.0, 57.2)
- added P0: Conn_01x01_Pin, Connector_Wire:SolderWire-0.1sqmm_1x01_D0.4mm_OD1mm, F.Cu at (141.8, 50.1)
- added P1: Conn_01x01_Pin, Connector_Wire:SolderWire-0.1sqmm_1x01_D0.4mm_OD1mm, F.Cu at (141.8, 46.8)
- added P1.5: Conn_01x01_Pin, Connector_Wire:SolderWire-0.1sqmm_1x01_D0.4mm_OD1mm, F.Cu at (144.5, 50.1)
- added P10: Conn_01x01_Pin, Connector_Wire:SolderWire-0.1sqmm_1x01_D0.4mm_OD1mm, F.Cu at (122.0, 61.8)
- added R3: 500, Capacitor_SMD:C_0805_2012Metric, F.Cu at (119.0, 39.0)
Connections:
- net +5V renamed LED_P
- net GND renamed LED_G
- U1 pad 1: LED -> Net-(U1-GPIO2_A0_D0)
- U1 pad 10: unconnected-(U1-GPIO9_D9_MISO-Pad10) -> Net-(G9-Pin_1)
- U1 pad 11: unconnected-(U1-GPIO10_D10_MOSI-Pad11) -> Net-(G10-Pin_1)
- U1 pad 3: unconnected-(U1-GPIO4_A2_D2-Pad3) -> Net-(G2-Pin_1)
- U1 pad 4: unconnected-(U1-GPIO5_A3_D3-Pad4) -> Net-(G3-Pin_1)
- U1 pad 7: unconnected-(U1-GPIO21_D6_TX-Pad7) -> Net-(G4-Pin_1)
- U1 pad 8: unconnected-(U1-GPIO20_D7_RX-Pad8) -> Net-(G7-Pin_1)
- U1 pad 9: unconnected-(U1-GPIO8_D8_SCK-Pad9) -> Net-(G8-Pin_1)
Routing:
- net Net-(G3-Pin_1): track 0.00 -> 19.5 mm
- net Net-(G2-Pin_1): track 0.00 -> 18.1 mm
- net Net-(G10-Pin_1): track 0.00 -> 13.6 mm
- net Net-(G8-Pin_1): track 0.00 -> 11.7 mm
- net +3.3V: track 0.00 -> 11.0 mm
- net Net-(G9-Pin_1): track 0.00 -> 10.2 mm
- net Net-(G7-Pin_1): track 0.00 -> 10.2 mm
- net Net-(G4-Pin_1): track 0.00 -> 7.50 mm
- net LED_P: track 233.1 -> 239.5 mm, vias 2 -> 1
- net Net-(BAT_P1-Pin_1): track 27.4 -> 33.1 mm
- net LED: track 8.57 -> 4.76 mm
- net Net-(U1-GPIO2_A0_D0): track 0.00 -> 3.21 mm
- net AS5600_ANALOG: track 36.3 -> 37.2 mm
- net Net-(D2-DOUT): track 11.6 -> 12.1 mm
- net Net-(D11-DOUT): track 11.6 -> 12.1 mm
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
Commit message: update
Parts:
- added LED_JUMP1: Jumper_2_Bridged, Jumper:SolderJumper-2_P1.3mm_Bridged2Bar_Pad1.0x1.5mm, F.Cu at (107.3, 70.0)
- added MAG_POWER1: Jumper_2_Bridged, Jumper:SolderJumper-2_P1.3mm_Bridged2Bar_Pad1.0x1.5mm, F.Cu at (120.3, 70.0)
- BAT_N1, BAT_P1: footprint Connector_Wire:SolderWire-0.1sqmm_1x01_D0.4mm_OD1mm -> Connector_Wire:SolderWire-0.5sqmm_1x01_D0.9mm_OD2.1mm
- C10, C11, C12, C13, C2, C3, C4, C5, C6, C7, C8, C9, D1, D10, D11, D12, D2, D3, D4, D5, D6, D7, D8, D9: moved to F.Cu
- G10, G2, G3, G4, G7, G8, G9, P0, P1, P1.5, P10, U1: moved to B.Cu
- moved D1 60.0 mm to (160.0, 70.0)
- moved D7 60.0 mm to (100.0, 70.0)
- moved C2 59.1 mm to (100.5, 64.8), turned to -10 degrees
- moved C8 59.1 mm to (159.5, 75.2), turned to 170 degrees
- moved C13 56.4 mm to (101.8, 80.3), turned to 20 degrees
- moved C7 56.4 mm to (158.2, 59.7), turned to -160 degrees
- moved D12 52.0 mm to (156.0, 55.0), turned to 120 degrees
- moved D2 52.0 mm to (156.0, 85.0), turned to 60 degrees
- moved D6 52.0 mm to (104.0, 85.0), turned to -60 degrees
- moved D8 52.0 mm to (104.0, 55.0), turned to -120 degrees
- moved C3 46.0 mm to (107.0, 50.7), turned to -40 degrees
- moved C9 46.0 mm to (153.0, 89.3), turned to 140 degrees
- moved C12 38.6 mm to (110.7, 93.0), turned to 50 degrees
- moved C6 38.6 mm to (149.3, 47.0), turned to -130 degrees
- moved D11 30.0 mm to (145.0, 44.0), turned to 150 degrees
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Connections:
- net Net-(BAT_P1-Pin_1) renamed BAT_P
- C1 pad 1: LED_P -> Net-(MAG_POWER1-B)
- P1 pad 1: LED_P -> +5V
- R1 pad 1: LED_P -> Net-(MAG_POWER1-B)
- R2 pad 2: LED_P -> Net-(MAG_POWER1-B)
- U1 pad 14: LED_P -> +5V
- U2 pad 1: LED_P -> Net-(MAG_POWER1-B)
Routing:
- net +5V: track 0.00 -> 48.1 mm
- net LED_P: track 239.5 -> 195.0 mm, vias 1 -> 0
- net Net-(MAG_POWER1-B): track 0.00 -> 32.4 mm
- net LED_G: track 18.6 -> 11.2 mm
- net BAT_P: track 33.1 -> 37.8 mm
- net AS5600_SCL: track 28.3 -> 24.1 mm, vias 0 -> 1
- net AS5600_SDA: track 33.5 -> 29.5 mm, vias 0 -> 1
- net LED: track 4.76 -> 3.71 mm, vias 1 -> 0
- net Net-(U1-GPIO2_A0_D0): track 3.21 -> 4.26 mm, vias 0 -> 1
- net AS5600_ANALOG: track 37.2 -> 38.0 mm, vias 0 -> 1
Other:
- board text added: "3V"
- board text added: "5v"
- board text added: "BATT_N"
- board text added: "BATT_P"
- board text added: "G10"
- board text added: "G2"
- board text added: "G3"
- board text added: "G4"
- board text added: "G7"
- board text added: "G8"
- board text added: "G9"
- board text added: "GND"
- board text added: "LED_POWER"
- board text added: "SENSOR_POWER"

Commit message: update
Other:
- board text added: "JLCJLCJLCJLC"
Changed lines of the file:
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@@
+		)
+	)
+	(gr_text "JLCJLCJLCJLC"
+		(at 135.5 82.25 0)
+		(layer "B.SilkS")
+		(effects
+			(font
+				(size 1 1)
+				(thickness 0.1)
+			)
+			(justify left bottom mirror)
 		)
 	)
